Commit message: Simple KR6 update

File: models/kuka_kr6_r900/urdf/kuka_kr6_r900_extrusion_simple.urdf (robot description, URDF)
Before this commit: robot kr6_r900_workspace, 11 links, 10 joints
Links:
- link eef_base_link: geometry collision mesh filename=../meshes/mini_hotend/collision/mini_hotend_collision.stl scale=.001 .001 .001; visual mesh filename=../meshes/mini_hotend/visual/mini_hotend_visual.stl scale=.001 .001 .001
Joints:
- joint eef_base_to_tcp: origin xyz=0.150539 0.001052 0.119157 rpy=0.0 1.57079632679 0.0 -> xyz=0.136569 0.008654 0.109056 rpy=0.0 1.57079632679 0.0
